Commit message: changes

File: opendog_description/ros2_control/ros2_control.xacro (robot description, xacro)
@@ -8,59 +8,264 @@
             <param name="imu_mounting_deg.roll">0</param>
         </hardware>
-        <joint name="left_hip_motor_joint">
-            <command_interface name="position"/>
-            <state_interface name="position"/>
-            <state_interface name="velocity"/>
-            <param name="can_channel">1</param>
+        <joint name="FL_hip_joint">
+            <command_interface name="position"/>
+            <state_interface name="position"/>
+            <state_interface name="velocity"/>
+            <param name="can_channel">2</param>
             <param name="can_id">1</param>
+            <param name="position_offset">0.45</param>
+            <param name="control_mode">position</param>
+        </joint>
+        <joint name="FL_uleg_joint">
+            <command_interface name="position"/>
+            <state_interface name="position"/>
+            <state_interface name="velocity"/>
+            <param name="can_channel">2</param>
+            <param name="can_id">2</param>
+            <param name="position_offset">-0.4</param>
+            <param name="control_mode">position</param>
+        </joint>
+        <joint name="FL_lleg_joint">
+            <command_interface name="position"/>
+            <state_interface name="position"/>
+            <state_interface name="velocity"/>
+            <param name="can_channel">2</param>
+            <param name="can_id">3</param>
+            <param name="position_offset">0.4</param>
+            <param name="control_mode">position</param>
+        </joint>
+        <joint name="FR_hip_joint">
+            <command_interface name="position"/>
+            <state_interface name="position"/>
+            <state_interface name="velocity"/>
+            <param name="can_channel">2</param>
+            <param name="can_id">4</param>
+            <param name="position_offset">-0.3</param>
+            <param name="control_mode">position</param>
+        </joint>
+        <joint name="FR_uleg_joint">
+            <command_interface name="position"/>
+            <state_interface name="position"/>
+            <state_interface name="velocity"/>
+            <param name="can_channel">2</param>
+            <param name="can_id">5</param>
+            <param name="position_offset">-0.0</param>
+            <param name="control_mode">position</param>
+        </joint>
+        <joint name="FR_lleg_joint">
+            <command_interface name="position"/>
+            <state_interface name="position"/>
+            <state_interface name="velocity"/>
+            <param name="can_channel">2</param>
+            <param name="can_id">6</param>
             <param name="position_offset">0.0</param>
             <param name="control_mode">position</param>
         </joint>
-        <joint name="left_knee_joint">
-            <command_interface name="position"/>
-            <state_interface name="position"/>
-            <state_interface name="velocity"/>
-            <param name="can_channel">1</param>
+        <joint name="BL_hip_joint">
+            <command_interface name="position"/>
+            <state_interface name="position"/>
+            <state_interface name="velocity"/>
+            <param name="can_channel">3</param>
+            <param name="can_id">7</param>
+            <param name="position_offset">-0.4</param>
+            <param name="control_mode">position</param>
+        </joint>
+        <joint name="BL_uleg_joint">
+            <command_interface name="position"/>
+            <state_interface name="position"/>
+            <state_interface name="velocity"/>
+            <param name="can_channel">3</param>
+            <param name="can_id">8</param>
+            <param name="position_offset">-0.3</param>
+            <param name="control_mode">position</param>
+        </joint>
+        <joint name="BL_lleg_joint">
+            <command_interface name="position"/>
+            <state_interface name="position"/>
+            <state_interface name="velocity"/>
+            <param name="can_channel">3</param>
+            <param name="can_id">9</param>
+            <param name="position_offset">-0.4</param>
+            <param name="control_mode">position</param>
+        </joint>
+        <joint name="BR_hip_joint">
+            <command_interface name="position"/>
+            <state_interface name="position"/>
+            <state_interface name="velocity"/>
+            <param name="can_channel">4</param>
+            <param name="can_id">10</param>
+            <param name="position_offset">0.4</param>
+            <param name="control_mode">position</param>
+        </joint>
+        <joint name="BR_uleg_joint">
+            <command_interface name="position"/>
+            <state_interface name="position"/>
+            <state_interface name="velocity"/>
+            <param name="can_channel">4</param>
+            <param name="can_id">11</param>
+            <param name="position_offset">-0.0</param>
+            <param name="control_mode">position</param>
+        </joint>
+        <joint name="BR_lleg_joint">
+            <command_interface name="position"/>
+            <state_interface name="position"/>
+            <state_interface name="velocity"/>
+            <param name="can_channel">4</param>
+            <param name="can_id">12</param>
+            <param name="position_offset">-0.4</param>
+            <param name="control_mode">position</param>
+        </joint>
+        <!--  -->
+        <!-- <joint name="FL_hip_joint">
+            <command_interface name="position">
+                <param name="min">-1.57</param>
+                <param name="max">1.57</param>
+            </command_interface>
+            <state_interface name="position">
+                <param name="initial_value">-0.0</param>
+            </state_interface>
+            <state_interface name="velocity"/>
+            <param name="can_channel">2</param>
+            <param name="can_id">1</param>
+            <param name="position_offset">-0.0</param>
+            <param name="control_mode">position</param>
+        </joint>
+        <joint name="FL_uleg_joint">
+            <command_interface name="position">
+                <param name="min">-1.2217</param>
+                <param name="max">3.14</param>
+            </command_interface>
+            <state_interface name="position">
+                <param name="initial_value">-0.0</param>
+            </state_interface>
+            <state_interface name="velocity"/>
+            <param name="can_channel">2</param>
             <param name="can_id">2</param>
             <param name="position_offset">-0.0</param>
             <param name="control_mode">position</param>
         </joint>
-        <!-- <joint name="left_wheel_joint">
-            <command_interface name="effort"/>
-            <state_interface name="position"/>
-            <state_interface name="velocity"/>
-            <param name="can_channel">1</param>
+        <joint name="FL_lleg_joint">
+            <command_interface name="position">
+                <param name="min">0.45</param>
+                <param name="max">2.3562</param>
+            </command_interface>
+            <state_interface name="position">
+                <param name="initial_value">0.45</param>
+            </state_interface>
+            <state_interface name="velocity"/>
+            <param name="can_channel">2</param>
             <param name="can_id">3</param>
-            <param name="position_offset">-0.1</param>
-            <param name="control_mode">effort</param>
+            <param name="position_offset">-0.0</param>
+            <param name="control_mode">position</param>
+        </joint>
+        <joint name="FR_hip_joint">
+            <command_interface name="position">
+                <param name="min">-1.57</param>
+                <param name="max">1.57</param>
+            </command_interface>
+            <state_interface name="position"/>
+            <state_interface name="velocity"/>
+            <param name="can_channel">2</param>
+            <param name="can_id">4</param>
+            <param name="position_offset">-0.0</param>
+            <param name="control_mode">position</param>
+        </joint>
+        <joint name="FR_uleg_joint">
+            <command_interface name="position">
+                <param name="min">-1.2217</param>
+                <param name="max">3.14</param>
+            </command_interface>
+            <state_interface name="position"/>
+            <state_interface name="velocity"/>
+            <param name="can_channel">2</param>
+            <param name="can_id">5</param>
+            <param name="position_offset">-0.0</param>
+            <param name="control_mode">position</param>
+        </joint>
+        <joint name="FR_lleg_joint">
+            <command_interface name="position">
+                <param name="min">0.45</param>
+                <param name="max">2.3562</param>
+            </command_interface>
+            <state_interface name="position"/>
+            <state_interface name="velocity"/>
+            <param name="can_channel">2</param>
+            <param name="can_id">6</param>
+            <param name="position_offset">0.45</param>
+            <param name="control_mode">position</param>
+        </joint>
+        <joint name="BL_hip_joint">
+            <command_interface name="position">
+                <param name="min">-1.57</param>
+                <param name="max">1.57</param>
+            </command_interface>
+            <state_interface name="position"/>
+            <state_interface name="velocity"/>
+            <param name="can_channel">3</param>
+            <param name="can_id">7</param>
+            <param name="position_offset">-0.0</param>
+            <param name="control_mode">position</param>
+        </joint>
+        <joint name="BL_uleg_joint">
+            <command_interface name="position">
+                <param name="min">-1.2217</param>
+                <param name="max">3.14</param>
+            </command_interface>
+            <state_interface name="position"/>
+            <state_interface name="velocity"/>
+            <param name="can_channel">3</param>
+            <param name="can_id">8</param>
+            <param name="position_offset">-0.0</param>
+            <param name="control_mode">position</param>
+        </joint>
+        <joint name="BL_lleg_joint">
+            <command_interface name="position">
+                <param name="min">0.45</param>
+                <param name="max">2.3562</param>
+            </command_interface>
+            <state_interface name="position"/>
+            <state_interface name="velocity"/>
+            <param name="can_channel">3</param>
+            <param name="can_id">9</param>
+            <param name="position_offset">0.45</param>
+            <param name="control_mode">position</param>
+        </joint>
+        <joint name="BR_hip_joint">
+            <command_interface name="position">
+                <param name="min">-1.57</param>
+                <param name="max">1.57</param>
+            </command_interface>
+            <state_interface name="position"/>
+            <state_interface name="velocity"/>
+            <param name="can_channel">4</param>
+            <param name="can_id">10</param>
+            <param name="position_offset">-0.0</param>
+            <param name="control_mode">position</param>
+        </joint>
+        <joint name="BR_uleg_joint">
+            <command_interface name="position">
+                <param name="min">-1.2217</param>
+                <param name="max">3.14</param>
+            </command_interface>
+            <state_interface name="position"/>
+            <state_interface name="velocity"/>
+            <param name="can_channel">4</param>
+            <param name="can_id">11</param>
+            <param name="position_offset">-0.0</param>
+            <param name="control_mode">position</param>
+        </joint>
+        <joint name="BR_lleg_joint">
+            <command_interface name="position">
+                <param name="min">0.45</param>
+                <param name="max">2.3562</param>
+            </command_interface>
+            <state_interface name="position"/>
+            <state_interface name="velocity"/>
+            <param name="can_channel">4</param>
+            <param name="can_id">12</param>
+            <param name="position_offset">0.45</param>
+            <param name="control_mode">position</param>
         </joint> -->
-        <joint name="right_hip_motor_joint">
-            <command_interface name="position"/>
-            <state_interface name="position"/>
-            <state_interface name="velocity"/>
-            <param name="can_channel">2</param>
-            <param name="can_id">4</param>
-            <param name="position_offset">0</param>
-            <param name="control_mode">position</param>
-        </joint>
-        <joint name="right_knee_joint">
-            <command_interface name="position"/>
-            <state_interface name="position"/>
-            <state_interface name="velocity"/>
-            <param name="can_channel">2</param>
-            <param name="can_id">5</param>
-            <param name="position_offset">0.0</param>
-            <param name="control_mode">position</param>
-        </joint>
-        <!-- <joint name="right_wheel_joint">
-            <command_interface name="effort"/>
-            <state_interface name="position"/>
-            <state_interface name="velocity"/>
-            <param name="can_channel">2</param>
-            <param name="can_id">6</param>
-            <param name="position_offset">-0.0</param>
-            <param name="control_mode">effort</param>
-        </joint> -->
-    <sensor name="imu_sensor">
+    <!-- <sensor name="imu_sensor">
         <state_interface name="orientation.x"/>
         <state_interface name="orientation.y"/>
@@ -73,5 +278,5 @@
         <state_interface name="linear_acceleration.y"/>
         <state_interface name="linear_acceleration.z"/>
-    </sensor>
+    </sensor> -->
     </ros2_control>
 </robot>

File: opendog_description/urdf/lidar.xacro (robot description, xacro)
@@ -15,5 +15,5 @@
     <!-- Output -->
     <odometry_frame>odom</odometry_frame>
-    <robot_base_frame>base_link</robot_base_frame>
+    <robot_base_frame>base_footprint</robot_base_frame>
     <publish_odom>true</publish_odom>
     <publish_odom_tf>true</publish_odom_tf>

File: opendog_description/urdf/opendog_joints.xacro (robot description, xacro)
@@ -6,4 +6,9 @@
         <parent link="base_link"/>
         <child link="world"/>
+    </joint>
+    <joint name="base_footprint_joint" type="fixed">
+        <parent link="base_link"/>
+        <child link="base_footprint"/>
+        <origin xyz="0 0 0" rpy="0 0 0"/>
     </joint>
     <!-- *********  FR_hip joint ********* -->

File: opendog_description/urdf/opendog_links.xacro (robot description, xacro)
@@ -45,4 +45,7 @@
         </collision>
     </link>
+<!-- *********** base footprint *********** -->
+    <link name="base_footprint">
+    </link>
     <!-- !!!!!!!!!!!!!!!!!!!!!!! HIPS !!!!!!!!!!!!!!!!!!!!!!!!!!!! -->
     <!-- *********** FR_hip *********** -->
